Commit message: rename project

File: robots/robot/hera_base.urdf.xacro (robot description, xacro)
@@ -10,15 +10,15 @@
   <!-- ##################################################################### -->
   <!-- commons -->
-  <xacro:include filename="$(find vault)/robots/urdf/commons.urdf.xacro" />
+  <xacro:include filename="$(find reinforcement-navigation)/robots/urdf/commons.urdf.xacro" />
   <!-- actuators -->
-  <xacro:include filename="$(find vault)/robots/urdf/actuators/base.urdf.xacro" />
+  <xacro:include filename="$(find reinforcement-navigation)/robots/urdf/actuators/base.urdf.xacro" />
   <!-- sensors -->
-  <xacro:include filename="$(find vault)/robots/urdf/sensors/hokuyo_utm.urdf.xacro"/>
-  <xacro:include filename="$(find vault)/robots/urdf/sensors/hokuyo_urg.urdf.xacro"/>
+  <xacro:include filename="$(find reinforcement-navigation)/robots/urdf/sensors/hokuyo_utm.urdf.xacro"/>
+  <xacro:include filename="$(find reinforcement-navigation)/robots/urdf/sensors/hokuyo_urg.urdf.xacro"/>
   <!-- simulation -->
-  <xacro:include filename="$(find vault)/robots/urdf/simulation/control.gazebo.xacro" />
-  <xacro:include filename="$(find vault)/robots/urdf/simulation/base.gazebo.xacro"/>
-  <xacro:include filename="$(find vault)/robots/urdf/simulation/hokuyo_utm.gazebo.xacro" />
-  <xacro:include filename="$(find vault)/robots/urdf/simulation/hokuyo_urg.gazebo.xacro" />
+  <xacro:include filename="$(find reinforcement-navigation)/robots/urdf/simulation/control.gazebo.xacro" />
+  <xacro:include filename="$(find reinforcement-navigation)/robots/urdf/simulation/base.gazebo.xacro"/>
+  <xacro:include filename="$(find reinforcement-navigation)/robots/urdf/simulation/hokuyo_utm.gazebo.xacro" />
+  <xacro:include filename="$(find reinforcement-navigation)/robots/urdf/simulation/hokuyo_urg.gazebo.xacro" />
 <!-- ####################################################################### -->
 <!-- ######################## robot parts ################################## -->

File: robots/urdf/actuators/base.urdf.xacro (robot description, xacro)
@@ -49,5 +49,5 @@
         <material name="black"/>
         <geometry>
-          <mesh filename="package://vault/robots/meshes/base.stl"/>
+          <mesh filename="package://reinforcement-navigation/robots/meshes/base.stl"/>
         </geometry>
       </visual>
@@ -62,5 +62,5 @@
         <material name="white"/>
         <geometry>
-          <mesh filename="package://vault/robots/meshes/wheelF.stl"/>
+          <mesh filename="package://reinforcement-navigation/robots/meshes/wheelF.stl"/>
         </geometry>
       </visual>
@@ -75,5 +75,5 @@
         <material name="white"/>
         <geometry>
-          <mesh filename="package://vault/robots/meshes/wheelF.stl"/>
+          <mesh filename="package://reinforcement-navigation/robots/meshes/wheelF.stl"/>
         </geometry>
       </visual>
@@ -88,5 +88,5 @@
         <material name="white"/>
         <geometry>
-          <mesh filename="package://vault/robots/meshes/wheelB.stl"/>
+          <mesh filename="package://reinforcement-navigation/robots/meshes/wheelB.stl"/>
         </geometry>
       </visual>
@@ -101,5 +101,5 @@
         <material name="white"/>
         <geometry>
-          <mesh filename="package://vault/robots/meshes/wheelB.stl"/>
+          <mesh filename="package://reinforcement-navigation/robots/meshes/wheelB.stl"/>
         </geometry>
       </visual>

File: robots/urdf/sensors/hokuyo_urg.urdf.xacro (robot description, xacro)
@@ -17,5 +17,5 @@
         <origin xyz="0 0 0" rpy="0 0 0" />
         <geometry>
-          <mesh filename="package://vault/robots/meshes/hokuyo_urg.dae" />
+          <mesh filename="package://reinforcement-navigation/robots/meshes/hokuyo_urg.dae" />
         </geometry>
       </visual>

File: robots/urdf/sensors/hokuyo_utm.urdf.xacro (robot description, xacro)
@@ -17,5 +17,5 @@
         <origin xyz="0 0 0" rpy="${M_PI/2} 0 0" />
         <geometry>
-          <mesh filename="package://vault/robots/meshes/hokuyo_utm.stl"/>
+          <mesh filename="package://reinforcement-navigation/robots/meshes/hokuyo_utm.stl"/>
         </geometry>
       </visual>

Commit message: rename project

File: robots/robot/hera_base.urdf.xacro (robot description, xacro)
@@ -10,15 +10,15 @@
   <!-- ##################################################################### -->
   <!-- commons -->
-  <xacro:include filename="$(find reinforcement-navigation)/robots/urdf/commons.urdf.xacro" />
+  <xacro:include filename="$(find reinforcement)/robots/urdf/commons.urdf.xacro" />
   <!-- actuators -->
-  <xacro:include filename="$(find reinforcement-navigation)/robots/urdf/actuators/base.urdf.xacro" />
+  <xacro:include filename="$(find reinforcement)/robots/urdf/actuators/base.urdf.xacro" />
   <!-- sensors -->
-  <xacro:include filename="$(find reinforcement-navigation)/robots/urdf/sensors/hokuyo_utm.urdf.xacro"/>
-  <xacro:include filename="$(find reinforcement-navigation)/robots/urdf/sensors/hokuyo_urg.urdf.xacro"/>
+  <xacro:include filename="$(find reinforcement)/robots/urdf/sensors/hokuyo_utm.urdf.xacro"/>
+  <xacro:include filename="$(find reinforcement)/robots/urdf/sensors/hokuyo_urg.urdf.xacro"/>
   <!-- simulation -->
-  <xacro:include filename="$(find reinforcement-navigation)/robots/urdf/simulation/control.gazebo.xacro" />
-  <xacro:include filename="$(find reinforcement-navigation)/robots/urdf/simulation/base.gazebo.xacro"/>
-  <xacro:include filename="$(find reinforcement-navigation)/robots/urdf/simulation/hokuyo_utm.gazebo.xacro" />
-  <xacro:include filename="$(find reinforcement-navigation)/robots/urdf/simulation/hokuyo_urg.gazebo.xacro" />
+  <xacro:include filename="$(find reinforcement)/robots/urdf/simulation/control.gazebo.xacro" />
+  <xacro:include filename="$(find reinforcement)/robots/urdf/simulation/base.gazebo.xacro"/>
+  <xacro:include filename="$(find reinforcement)/robots/urdf/simulation/hokuyo_utm.gazebo.xacro" />
+  <xacro:include filename="$(find reinforcement)/robots/urdf/simulation/hokuyo_urg.gazebo.xacro" />
 <!-- ####################################################################### -->
 <!-- ######################## robot parts ################################## -->

File: robots/urdf/actuators/base.urdf.xacro (robot description, xacro)
@@ -49,5 +49,5 @@
         <material name="black"/>
         <geometry>
-          <mesh filename="package://reinforcement-navigation/robots/meshes/base.stl"/>
+          <mesh filename="package://reinforcement/robots/meshes/base.stl"/>
         </geometry>
       </visual>
@@ -62,5 +62,5 @@
         <material name="white"/>
         <geometry>
-          <mesh filename="package://reinforcement-navigation/robots/meshes/wheelF.stl"/>
+          <mesh filename="package://reinforcement/robots/meshes/wheelF.stl"/>
         </geometry>
       </visual>
@@ -75,5 +75,5 @@
         <material name="white"/>
         <geometry>
-          <mesh filename="package://reinforcement-navigation/robots/meshes/wheelF.stl"/>
+          <mesh filename="package://reinforcement/robots/meshes/wheelF.stl"/>
         </geometry>
       </visual>
@@ -88,5 +88,5 @@
         <material name="white"/>
         <geometry>
-          <mesh filename="package://reinforcement-navigation/robots/meshes/wheelB.stl"/>
+          <mesh filename="package://reinforcement/robots/meshes/wheelB.stl"/>
         </geometry>
       </visual>
@@ -101,5 +101,5 @@
         <material name="white"/>
         <geometry>
-          <mesh filename="package://reinforcement-navigation/robots/meshes/wheelB.stl"/>
+          <mesh filename="package://reinforcement/robots/meshes/wheelB.stl"/>
         </geometry>
       </visual>

File: robots/urdf/sensors/hokuyo_urg.urdf.xacro (robot description, xacro)
@@ -17,5 +17,5 @@
         <origin xyz="0 0 0" rpy="0 0 0" />
         <geometry>
-          <mesh filename="package://reinforcement-navigation/robots/meshes/hokuyo_urg.dae" />
+          <mesh filename="package://reinforcement/robots/meshes/hokuyo_urg.dae" />
         </geometry>
       </visual>

File: robots/urdf/sensors/hokuyo_utm.urdf.xacro (robot description, xacro)
@@ -17,5 +17,5 @@
         <origin xyz="0 0 0" rpy="${M_PI/2} 0 0" />
         <geometry>
-          <mesh filename="package://reinforcement-navigation/robots/meshes/hokuyo_utm.stl"/>
+          <mesh filename="package://reinforcement/robots/meshes/hokuyo_utm.stl"/>
         </geometry>
       </visual>
